File: demodulator.kicad_sch (KiCad schematic)
At the start: 12 parts, among them J1 Input, J2 Output, U1 MAX941xPA, U2 MAX941xPA

Commit message: PCB design
Parts:
- removed J1: Input, symbol Connector:Conn_01x01_Pin
- removed J2: Output, symbol Connector:Conn_01x01_Pin
- removed U1, U2: MAX941xPA, Package_DIP:DIP-8_W7.62mm, symbol Comparator:MAX941xPA
- added C3: 1u, Capacitor_SMD:C_0805_2012Metric_Pad1.18x1.45mm_HandSolder, symbol Device:C
- added H1, H2, H3, H4: MountingHole_Pad, MountingHole:MountingHole_2.2mm_M2_ISO14580_Pad, symbol Mechanical:MountingHole_Pad
- added J1: Conn_01x02, Connector_Samtec_HPM_THT:Samtec_HPM-02-05-x-S_Straight_1x02_Pitch5.08mm, symbol Connector_Generic:Conn_01x02
- added J4: Conn_01x16, Connector_PinSocket_2.54mm:PinSocket_1x16_P2.54mm_Vertical, symbol Connector_Generic:Conn_01x16
- added J5: Conn_01x12, Connector_PinSocket_2.54mm:PinSocket_1x12_P2.54mm_Vertical, symbol Connector_Generic:Conn_01x12
- added U1: MAX942, Package_SO:SOIC-8_3.9x4.9mm_P1.27mm, symbol components:MAX942
- C1, C2: footprint (none) -> Capacitor_SMD:C_0805_2012Metric_Pad1.18x1.45mm_HandSolder
- D1: footprint (none) -> Diode_SMD:D_0805_2012Metric_Pad1.15x1.40mm_HandSolder
- R1, R2, R3: footprint (none) -> Resistor_SMD:R_0805_2012Metric_Pad1.20x1.40mm_HandSolder
- RV1, RV2: footprint (none) -> Potentiometer_SMD:Potentiometer_Bourns_TC33X_Vertical
Connections:
- net GND: now also C3.1, H1.1, H2.1, H3.1, H4.1, J1.2 (Pin_2), J4.16 (Pin_16), J4.4 (Pin_4), U1.4 (V-)
- net at C1.1, D1.1 (K), R1.1: now also U1.6 (-)
- net at C2.2, R2.2, R3.1: now also U1.3 (+)
- net at RV1.2: now also U1.2 (-)
- net at RV2.2: now also U1.5 (+)
- net at D1.2 (A): now also U1.1
- net at C2.1: now also J1.1 (Pin_1)
- net +5V renamed +3.3V
- net +3.3V: now also C3.2, J4.2 (Pin_2), U1.8 (V+)
- new net TX: J4.14 (Pin_14), U1.7
- no-connect marks 0 -> 24
